File: swing-atreus.kicad_pcb (KiCad board)
At the start: 2 copper layers, 131 x 109.8 mm, 81 parts, among them J1 Conn_01x02_Female, SW1 SW_SPDT, SW10 SW_SPST, SW11 SW_SPST, SW12 SW_SPST, SW13 SW_SPST, SW14 SW_SPST, SW15 SW_SPST, SW16 SW_SPST, SW17 SW_SPST, SW18 SW_SPST, SW19 SW_SPST, SW20 SW_SPST, SW21 SW_SPST, SW22 SW_SPST, SW23 SW_SPST, SW24 SW_SPST, SW25 SW_SPST, SW26 SW_SPST, SW27 SW_SPST, SW28 SW_SPST, SW29 SW_SPST, SW3 SW_SPST, SW30 SW_SPST, SW31 SW_SPST, SW32 SW_SPST, SW33 SW_SPST, SW34 SW_SPST, SW4 SW_SPST, SW5 SW_SPST, SW6 SW_SPST, SW7 SW_SPST, SW8 SW_SPST, SW9 SW_SPST, U1 nice!nano

Commit message: update to single board design
Parts:
- removed GND select: SolderJumper-3_P1.3mm_Open_Pad1.0x1.5mm, Jumper:SolderJumper-3_P1.3mm_Open_Pad1.0x1.5mm
- removed the J1 at (157.1, 77.9)
- removed REF** (x11): MountingHole_2.5mm, MountingHole:MountingHole_2.5mm
- removed power select: SolderJumper-3_P1.3mm_Open_Pad1.0x1.5mm, Jumper:SolderJumper-3_P1.3mm_Open_Pad1.0x1.5mm
- added D33: D0, Diode_SMD:D_SOD-123, F.Cu at (241.4, 82.7)
- added D34: D0, Diode_SMD:D_SOD-123, F.Cu at (245.0, 101.2)
- added D35: D0, Diode_SMD:D_SOD-123, F.Cu at (248.6, 119.9)
- added D36: D0, Diode_SMD:D_SOD-123, F.Cu at (252.0, 138.6)
- added D37: D0, Diode_SMD:D_SOD-123, F.Cu at (255.7, 157.1)
- added D38: D0, Diode_SMD:D_SOD-123, F.Cu at (259.2, 73.7)
- added D39: D0, Diode_SMD:D_SOD-123, F.Cu at (262.6, 92.8)
- added D40: D0, Diode_SMD:D_SOD-123, F.Cu at (266.3, 111.2)
- added D41: D0, Diode_SMD:D_SOD-123, F.Cu at (269.8, 130.2)
- added D42: D0, Diode_SMD:D_SOD-123, F.Cu at (273.4, 148.3)
- added D43: D0, Diode_SMD:D_SOD-123, F.Cu at (277.1, 65.5)
- added D44: D0, Diode_SMD:D_SOD-123, F.Cu at (280.7, 84.1)
- added D45: D0, Diode_SMD:D_SOD-123, F.Cu at (284.1, 103.0)
- added D46: D0, Diode_SMD:D_SOD-123, F.Cu at (287.7, 122.1)
- added D47: D0, Diode_SMD:D_SOD-123, F.Cu at (291.2, 141.4)
- added D48: D0, Diode_SMD:D_SOD-123, F.Cu at (296.3, 66.7)
- added D49: D0, Diode_SMD:D_SOD-123, F.Cu at (299.4, 85.9)
- added D50: D0, Diode_SMD:D_SOD-123, F.Cu at (303.2, 104.7)
- added D51: D0, Diode_SMD:D_SOD-123, F.Cu at (307.0, 123.1)
- added D52: D0, Diode_SMD:D_SOD-123, F.Cu at (310.6, 141.7)
- added D53: D0, Diode_SMD:D_SOD-123, F.Cu at (316.1, 68.3)
- added D54: D0, Diode_SMD:D_SOD-123, F.Cu at (319.1, 86.9)
- added D55: D0, Diode_SMD:D_SOD-123, F.Cu at (323.0, 105.5)
- added D56: D0, Diode_SMD:D_SOD-123, F.Cu at (327.0, 124.3)
- added D57: D0, Diode_SMD:D_SOD-123, F.Cu at (330.1, 142.9)
- added D58: D0, Diode_SMD:D_SOD-123, F.Cu at (334.7, 64.8)
- added D59: D0, Diode_SMD:D_SOD-123, F.Cu at (337.7, 83.4)
- added D60: D0, Diode_SMD:D_SOD-123, F.Cu at (341.7, 101.9)
- added D61: D0, Diode_SMD:D_SOD-123, F.Cu at (345.2, 120.4)
- added D62: D0, Diode_SMD:D_SOD-123, F.Cu at (349.0, 139.2)
- added D63: D0, Diode_SMD:D_SOD-123, F.Cu at (231.7, 136.0)
- added D64: D0, Diode_SMD:D_SOD-123, F.Cu at (235.0, 154.3)
- added SW2: SW_SPST, PCM_Switch_Keyboard_Kailh:SW_Kailh_Choc_V1V2_double, F.Cu at (241.9, 92.2)
- added SW35: SW_SPST, PCM_Switch_Keyboard_Kailh:SW_Kailh_Choc_V1V2_double, F.Cu at (245.5, 110.9)
- added SW36: SW_SPST, PCM_Switch_Keyboard_Kailh:SW_Kailh_Choc_V1V2_double, F.Cu at (249.1, 129.5)
- added SW37: SW_SPST, PCM_Switch_Keyboard_Kailh:SW_Kailh_Choc_V1V2_double, F.Cu at (252.7, 148.2)
- added SW38: SW_SPST, PCM_Switch_Keyboard_Kailh:SW_Kailh_Choc_V1V2_double, F.Cu at (256.3, 166.9)
- added SW39: SW_SPST, PCM_Switch_Keyboard_Kailh:SW_Kailh_Choc_V1V2_double, F.Cu at (259.6, 83.7)
- added SW40: SW_SPST, PCM_Switch_Keyboard_Kailh:SW_Kailh_Choc_V1V2_double, F.Cu at (263.3, 102.2)
- added SW41: SW_SPST, PCM_Switch_Keyboard_Kailh:SW_Kailh_Choc_V1V2_double, F.Cu at (266.8, 120.9)
- added SW42: SW_SPST, PCM_Switch_Keyboard_Kailh:SW_Kailh_Choc_V1V2_double, F.Cu at (270.5, 139.7)
- added SW43: SW_SPST, PCM_Switch_Keyboard_Kailh:SW_Kailh_Choc_V1V2_double, F.Cu at (274.2, 158.2)
- added SW44: SW_SPST, PCM_Switch_Keyboard_Kailh:SW_Kailh_Choc_V1V2_double, F.Cu at (277.4, 75.2)
- added SW45: SW_SPST, PCM_Switch_Keyboard_Kailh:SW_Kailh_Choc_V1V2_double, F.Cu at (281.1, 93.9)
- added SW46: SW_SPST, PCM_Switch_Keyboard_Kailh:SW_Kailh_Choc_V1V2_double, F.Cu at (284.6, 112.6)
- added SW47: SW_SPST, PCM_Switch_Keyboard_Kailh:SW_Kailh_Choc_V1V2_double, F.Cu at (288.3, 131.7)
- added SW48: SW_SPST, PCM_Switch_Keyboard_Kailh:SW_Kailh_Choc_V1V2_double, F.Cu at (292.1, 151.2)
- added SW49: SW_SPST, PCM_Switch_Keyboard_Kailh:SW_Kailh_Choc_V1V2_double, F.Cu at (296.9, 76.5)
- added SW50: SW_SPST, PCM_Switch_Keyboard_Kailh:SW_Kailh_Choc_V1V2_double, F.Cu at (300.8, 95.3)
- added SW51: SW_SPST, PCM_Switch_Keyboard_Kailh:SW_Kailh_Choc_V1V2_double, F.Cu at (304.3, 114.3)
- added SW52: SW_SPST, PCM_Switch_Keyboard_Kailh:SW_Kailh_Choc_V1V2_double, F.Cu at (307.7, 132.6)
- added SW53: SW_SPST, PCM_Switch_Keyboard_Kailh:SW_Kailh_Choc_V1V2_double, F.Cu at (311.8, 151.2)
- added SW54: SW_SPST, PCM_Switch_Keyboard_Kailh:SW_Kailh_Choc_V1V2_double, F.Cu at (316.6, 77.9)
- added SW55: SW_SPST, PCM_Switch_Keyboard_Kailh:SW_Kailh_Choc_V1V2_double, F.Cu at (320.2, 96.5)
- added SW56: SW_SPST, PCM_Switch_Keyboard_Kailh:SW_Kailh_Choc_V1V2_double, F.Cu at (324.0, 115.2)
- added SW57: SW_SPST, PCM_Switch_Keyboard_Kailh:SW_Kailh_Choc_V1V2_double, F.Cu at (327.7, 133.9)
- added SW58: SW_SPST, PCM_Switch_Keyboard_Kailh:SW_Kailh_Choc_V1V2_double, F.Cu at (331.2, 152.5)
- added SW59: SW_SPST, PCM_Switch_Keyboard_Kailh:SW_Kailh_Choc_V1V2_double, F.Cu at (335.4, 74.2)
- added SW60: SW_SPST, PCM_Switch_Keyboard_Kailh:SW_Kailh_Choc_V1V2_double, F.Cu at (339.0, 92.9)
- added SW61: SW_SPST, PCM_Switch_Keyboard_Kailh:SW_Kailh_Choc_V1V2_double, F.Cu at (342.6, 111.2)
- added SW62: SW_SPST, PCM_Switch_Keyboard_Kailh:SW_Kailh_Choc_V1V2_double, F.Cu at (346.3, 130.3)
- added SW63: SW_SPST, PCM_Switch_Keyboard_Kailh:SW_Kailh_Choc_V1V2_double, F.Cu at (349.9, 148.8)
- added SW64: SW_SPST, PCM_Switch_Keyboard_Kailh:SW_Kailh_Choc_V1V2_double, F.Cu at (232.1, 145.4)
- added SW65: SW_SPST, PCM_Switch_Keyboard_Kailh:SW_Kailh_Choc_V1V2_double, F.Cu at (235.7, 164.0)
- SW10, SW11, SW12, SW13, SW14, SW15, SW16, SW17, SW18, SW19, SW20, SW21, SW22, SW23, SW24, SW25, SW26, SW27, SW28, SW29, SW3, SW30, SW31, SW32, SW33, SW34, SW4, SW5, SW6, SW7, SW8, SW9: footprint kailh:Kailh_low_profile -> PCM_Switch_Keyboard_Kailh:SW_Kailh_Choc_V1V2_double
- moved SW1 171.8 mm to (234.6, 62.0)
- moved D26 68.0 mm to (187.9, 82.4), turned to 169 degrees
- moved SW28 66.6 mm to (185.7, 91.2), turned to -11 degrees
- moved D21 65.8 mm to (170.2, 73.9), turned to 169 degrees
- moved D27 65.1 mm to (183.8, 100.5), turned to 169 degrees
- moved SW23 64.4 mm to (168.0, 82.6), turned to -11 degrees
- moved D16 63.8 mm to (152.5, 65.4), turned to 169 degrees
- moved SW29 63.8 mm to (182.0, 109.8), turned to -11 degrees
- moved J1 63.4 mm to (214.2, 100.8), turned to 0 degrees
- moved D22 62.9 mm to (166.7, 92.6), turned to 169 degrees
- moved D28 62.4 mm to (180.7, 119.2), turned to 169 degrees
- moved SW18 62.3 mm to (150.3, 74.1), turned to -11 degrees
- moved SW24 61.5 mm to (164.3, 101.3), turned to -11 degrees
- moved SW30 61.0 mm to (178.4, 128.5), turned to -11 degrees
- moved D17 60.8 mm to (148.9, 84.0), turned to 169 degrees
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Connections:
- net Net-(SW1-Pad2) renamed /VBAT
- J1 pad 1: Net-(J1-Pad1) -> GND
- J1 pad 2: GND -> Net-(J1-Pin_2)
- SW1 pad 1: Net-(SW1-Pad1) -> unconnected-(SW1-A-Pad1)
- SW1 pad 3: Net-(J1-Pad1) -> Net-(J1-Pin_2)
- U1 pad 1: Net-(U1-Pad1) -> /L_Row1
- U1 pad 10: Net-(U1-Pad10) -> /L_Row8
- U1 pad 11: Net-(U1-Pad11) -> /L_Row9
- U1 pad 12: Net-(U1-Pad12) -> /L_Row10
- U1 pad 13: Net-(U1-Pad13) -> unconnected-(U1-D10/P0.09-Pad13)
- U1 pad 2: Net-(U1-Pad2) -> /L_Row2
- U1 pad 21: Net-(U1-Pad21) -> unconnected-(U1-_3v3_(out)-Pad21)
- U1 pad 22: Net-(SW2-Pad1) -> unconnected-(U1-Reset-Pad22)
- U1 pad 23: Net-(U1-Pad23) -> unconnected-(U1-Gnd-Pad23)
- U1 pad 4: GND -> unconnected-(U1-GND-Pad4)
- U1 pad 5: /L_Row1 -> /L_Row3
- U1 pad 6: /L_Row2 -> /L_Row4
- U1 pad 7: /L_Row3 -> /L_Row5
- U1 pad 8: /L_Row4 -> /L_Row6
- U1 pad 9: /L_Row5 -> /L_Row7
Routing:
- net /L_Row10: track 0.00 -> 230.0 mm
- net /L_Row8: track 0.00 -> 226.9 mm, vias 0 -> 2
- net /L_Row7: track 0.00 -> 205.3 mm
- net /L_column6: track 117.7 -> 318.5 mm
- net /L_Row9: track 0.00 -> 191.8 mm, vias 0 -> 1
- net /L_column4: track 148.7 -> 337.9 mm, vias 4 -> 1
- net /L_column5: track 134.5 -> 320.5 mm
- net /L_column3: track 163.6 -> 344.2 mm, vias 2 -> 1
- net /L_column2: track 180.9 -> 344.6 mm, vias 2 -> 1
- net /L_column1: track 196.1 -> 355.3 mm, vias 2 -> 1
- net /L_Row6: track 0.00 -> 158.1 mm, vias 0 -> 2
- net Net-(J1-Pad1): track 155.7 -> 0.00 mm, vias 3 -> 0
- net /VBAT: track 115.1 -> 14.3 mm, vias 3 -> 0
- net /L_column7: track 48.1 -> 142.0 mm
- net /L_Row2: track 117.2 -> 166.9 mm
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- removed copper zone on B.Cu, net GND
Other:
- board size 131 x 109.8 mm -> 295.2 x 122.6 mm
- net class Default removed
- net class signal removed
- board text removed: "solder inboard for left hand towards edge for right hand"

Commit message: add copper fills
Routing:
- added copper zone on B.Cu, net GND
- added copper zone on F.Cu, net GND
Changed lines of the file:
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@@
     (pad_to_mask_clearance 0)
     (pcbplotparams
-      (layerselection 0x0001000_7ffffffe)
+      (layerselection 0x00310fc_ffffffff)
       (plot_on_all_layers_selection 0x0000000_00000000)
       (disableapertmacros false)
@@
       (sketchpadsonfab false)
       (subtractmaskfromsilk false)
-      (outputformat 5)
+      (outputformat 1)
       (mirror false)
-      (drillshape 2)
+      (drillshape 0)
       (scaleselection 1)
       (outputdirectory "gerbs/")
@@
     (pad "2" smd roundrect (at 1 -2.85) (size 1 3.5) (layers "F.Cu" "F.Paste" "F.Mask") (roundrect_rratio 0.25)
       (net 89 "Net-(J1-Pin_2)") (pinfunction "Pin_2") (pintype "passive"))
-    (pad "MP" smd roundrect (at -3.35 2.9) (size 1.5 3.4) (layers "F.Cu" "F.Paste" "F.Mask") (roundrect_rratio 0.166667))
-    (pad "MP" smd roundrect (at 3.35 2.9) (size 1.5 3.4) (layers "F.Cu" "F.Paste" "F.Mask") (roundrect_rratio 0.166667))
+    (pad "MP" smd roundrect (at -3.35 2.9) (size 1.5 3.4) (layers "F.Cu" "F.Paste" "F.Mask") (roundrect_rratio 0.1666673333))
+    (pad "MP" smd roundrect (at 3.35 2.9) (size 1.5 3.4) (layers "F.Cu" "F.Paste" "F.Mask") (roundrect_rratio 0.1666673333))
     (model "${KISYS3DMOD}/Connector_JST.3dshapes/JST_PH_S2B-PH-SM4-TB_1x02-1MP_P2.00mm_Horizontal.wrl"
       (offset (xyz 0 0 0))
@@
   (segment (start 191.428391 154.65111) (end 192.016215 155.238934) (width 0.2) (layer "F.Cu") (net 90))
   (segment (start 192.016215 155.238934) (end 192.016215 158.178072) (width 0.2) (layer "F.Cu") (net 90))
+  (zone (net 33) (net_name "GND") (layers "F&B.Cu") (hatch edge 0.5)
+    (connect_pads (clearance 0.508))
+    (min_thickness 0.25) (filled_areas_thickness no)
+    (fill yes (thermal_gap 0.5) (thermal_bridge_width 0.5))
+    (polygon
+      (pts
+        (xy 361.45 59.375)
+        (xy 65.925 59.15)
+        (xy 65.925 181.475)
+        (xy 361.925 183.075)
+      )
+    )
+  )
 )
